File: DET100A_amp_5V/DET100A_amp_5V.kicad_pcb (KiCad board)
At the start: 2 copper layers, 50 x 25 mm, 15 parts, among them J1 5227677-1, J2 Screw_Terminal_01x03, J3 5227677-1, U1 OPA656NB/250

Commit message: feat: add some silkscreen elements
Parts:
- moved C4 0.29 mm to (124.3, 85.2)
- moved C9 0.19 mm to (124.3, 87.3)
Other:
- board text added: "+5V"
- board text added: "-5V"
- board text added: "IN"
- board text added: "OUT"
Changed lines of the file:
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@@
 	(footprint "Capacitor_SMD:C_0805_2012Metric_Pad1.18x1.45mm_HandSolder"
 		(layer "F.Cu")
-		(at 124.341702 85.5 180)
+		(at 124.341702 85.208177 180)
 		(descr "Capacitor SMD 0805 (2012 Metric), square (rectangular) end terminal, IPC-7351 nominal with elongated pad for handsoldering. (Body size source: IPC-SM-782 page 76, https://www.pcb-3d.com/wordpress/wp-content/uploads/ipc-sm-782a_amendment_1_and_2.pdf, https://docs.google.com/spreadsheets/d/1BsfQQcO9C6DZCsRaXUlFlo91Tg2WpOkGARC1WS5S8t0/edit?usp=sharing)")
 		(tags "capacitor handsolder")
@@
 	(footprint "Capacitor_SMD:C_0805_2012Metric_Pad1.18x1.45mm_HandSolder"
 		(layer "F.Cu")
-		(at 124.341702 87.5)
+		(at 124.341702 87.310361)
 		(descr "Capacitor SMD 0805 (2012 Metric), square (rectangular) end terminal, IPC-7351 nominal with elongated pad for handsoldering. (Body size source: IPC-SM-782 page 76, https://www.pcb-3d.com/wordpress/wp-content/uploads/ipc-sm-782a_amendment_1_and_2.pdf, https://docs.google.com/spreadsheets/d/1BsfQQcO9C6DZCsRaXUlFlo91Tg2WpOkGARC1WS5S8t0/edit?usp=sharing)")
 		(tags "capacitor handsolder")
@@
 		(tags "THT Terminal Block TE 282834-3 pitch 2.54mm size 8.08x6.5mm drill 1.1mm pad 2.1mm")
 		(property "Reference" "J2"
-			(at -3 0 0)
+			(at 8 -2.5 0)
 			(layer "F.SilkS")
 			(effects
@@
 		(layer "Edge.Cuts")
 	)
+	(gr_text "-5V"
+		(at 110 96.5 0)
+		(layer "F.SilkS")
+		(effects
+			(font
+				(size 0.75 0.75)
+				(thickness 0.1)
+			)
+			(justify left bottom)
+		)
+	)
+	(gr_text "+5V"
+		(at 121.2 96.5 0)
+		(layer "F.SilkS")
+		(effects
+			(font
+				(size 0.75 0.75)
+				(thickness 0.1)
+			)
+			(justify left bottom)
+		)
+	)
 	(gr_text "Tokamak\nGOLEM"
 		(at 139.5 96.5 0)
@@
 				(thickness 0.1)
 			)
+			(justify left bottom)
+		)
+	)
+	(gr_text "IN"
+		(at 102.25 92.75 0)
+		(layer "F.SilkS")
+		(effects
+			(font
+				(size 1 1)
+				(thickness 0.1)
+			)
+			(justify left bottom)
+		)
+	)
+	(gr_text "OUT"
+		(at 145 92.75 0)
+		(layer "F.SilkS")
+		(effects
+			(font
+				(size 1 1)
+				(thickness 0.1)
+			)
