File: DET100A_amp_5V/DET100A_amp_5V-rezac.kicad_pcb (KiCad board)
At the start: 2 copper layers, 50 x 25 mm, 15 parts, among them J1 5227677-1, J2 Screw_Terminal_01x03, J3 5227677-1, U1 OPA656NB/250

Commit message: konzultace 18.6.2026, board, 3D print settings
Routing:
- net GND: track 175.7 -> 170.2 mm, vias 80 -> 66
